Commit message: Added ros control for revolute joints

File: r2b_description/urdf/r2b.xacro (robot description, xacro)
@@ -1,4 +1,5 @@
 <?xml version="1.0" encoding="utf-8"?>
-<robot name="r2b_description">
+<robot name="r2b_description" xmlns:xacro="http://www.ros.org/wiki/xacro">
+  <link name='world'/>
   <link
     name="base_link">
@@ -41,4 +42,9 @@
     </collision>
   </link>
+  <joint name="fixed" type="fixed">
+		<origin xyz="0.0 0.0 0.0" rpy="0.0 0.0 0.0"/>
+		<parent link="world"/>
+		<child link="base_link"/>
+	</joint>
   <link
     name="link_1">
@@ -157,3 +163,5 @@
       velocity="0" />
   </joint>
+  <xacro:include filename="$(find r2b_description)/urdf/r2b_gazebo.xacro"/>
+  <xacro:revolute_controllers/>
 </robot>
