Commit message: Enabled collision without contact for r2b

File: r2b_description/urdf/r2b_gazebo.xacro (robot description, xacro)
@@ -23,10 +23,34 @@
 		<gazebo reference="base_link">
 			<material>Gazebo/Blue</material>
+			<collision>
+				<surface>
+				<contact>
+					<collide_without_contact>true</collide_without_contact>
+				</contact>
+				</surface>
+			</collision>
+			<selfCollide>false</selfCollide>
 		</gazebo>
 		<gazebo reference="link_1">
 			<material>Gazebo/Red</material>
+			<collision>
+				<surface>
+				<contact>
+					<collide_without_contact>true</collide_without_contact>
+				</contact>
+				</surface>
+			</collision>
+			<selfCollide>false</selfCollide>
 		</gazebo>
 		<gazebo reference="link_2">
 			<material>Gazebo/Orange</material>
+			<collision>
+				<surface>
+				<contact>
+					<collide_without_contact>true</collide_without_contact>
+				</contact>
+				</surface>
+			</collision>
+			<selfCollide>false</selfCollide>
 		</gazebo>
 		<!-- ros control plugin -->
