Commit message: Changed ref frame for boxes

File: r2b_env/urdf/box_common.xacro (robot description, xacro)
@@ -5,7 +5,10 @@
 	<xacro:property name="z" value="0.028"/>
 	<xacro:property name="mass" value="0.03"/>
+	<xacro:macro name="offseted_origin">
+		<origin xyz="-${x/2} 0.0 0.0" rpy="0.0 0.0 0.0"/>
+	</xacro:macro>
 	<xacro:macro name="box_inertia" params="m x y z">
 		<inertial>
-			<origin xyz="0.0 0.0 0.0" rpy="0.0 0.0 0.0"/>
+			<xacro:offseted_origin/>
 			<mass value="${m}"/>
 			<inertia ixx="${m*(y*y+z*z)/12}" ixy="0.0" ixz="0.0"

File: r2b_env/urdf/box_down.urdf.xacro (robot description, xacro)
@@ -5,5 +5,5 @@
 		<xacro:box_inertia m="${mass}" x="${x}" y="${y}" z="${z}"/>
 		<visual>
-			<origin xyz="0.0 0.0 0.0" rpy="0.0 0.0 0.0"/>
+			<xacro:offseted_origin/>
 			<geometry>
 				<box size="${x} ${y} ${z}"/>
@@ -11,5 +11,5 @@
 		</visual>
 		<collision>
-			<origin xyz="0.0 0.0 0.0" rpy="0.0 0.0 0.0"/>
+			<xacro:offseted_origin/>
 			<geometry>
 				<box size="${x} ${y} ${z}"/>

File: r2b_env/urdf/box_mid.urdf.xacro (robot description, xacro)
@@ -5,5 +5,5 @@
 		<xacro:box_inertia m="${mass}" x="${x}" y="${y}" z="${z}"/>
 		<visual>
-			<origin xyz="0.0 0.0 0.0" rpy="0.0 0.0 0.0"/>
+			<xacro:offseted_origin/>
 			<geometry>
 				<box size="${x} ${y} ${z}"/>
@@ -11,5 +11,5 @@
 		</visual>
 		<collision>
-			<origin xyz="0.0 0.0 0.0" rpy="0.0 0.0 0.0"/>
+			<xacro:offseted_origin/>
 			<geometry>
 				<box size="${x} ${y} ${z}"/>

File: r2b_env/urdf/box_top.urdf.xacro (robot description, xacro)
@@ -5,5 +5,5 @@
 		<xacro:box_inertia m="${mass}" x="${x}" y="${y}" z="${z}"/>
 		<visual>
-			<origin xyz="0.0 0.0 0.0" rpy="0.0 0.0 0.0"/>
+			<xacro:offseted_origin/>
 			<geometry>
 				<box size="${x} ${y} ${z}"/>
@@ -11,5 +11,5 @@
 		</visual>
 		<collision>
-			<origin xyz="0.0 0.0 0.0" rpy="0.0 0.0 0.0"/>
+			<xacro:offseted_origin/>
 			<geometry>
 				<box size="${x} ${y} ${z}"/>

Commit message: Reduced mass of boxes to make it easier for lifting

File: r2b_env/urdf/box_common.xacro (robot description, xacro)
@@ -4,5 +4,5 @@
 	<xacro:property name="y" value="0.03"/>
 	<xacro:property name="z" value="0.028"/>
-	<xacro:property name="mass" value="0.03"/>
+	<xacro:property name="mass" value="0.0003"/>
 	<xacro:macro name="offseted_origin">
 		<origin xyz="-${x/2} 0.0 0.0" rpy="0.0 0.0 0.0"/>
