Commit message: Removed unnecessary comments

File: r2b_env/urdf/compartments.urdf.xacro (robot description, xacro)
@@ -105,162 +105,6 @@
       <material>Gazebo/Yellow</material>
   </gazebo>
-  <!-- <link
-    name="box_top">
-    <inertial>
-      <origin
-        xyz="-0.015 0 6.9389E-18"
-        rpy="0 0 0" />
-      <mass
-        value="0.030353" />
-      <inertia
-        ixx="5.2421E-06"
-        ixy="1.9222E-21"
-        ixz="-1.5064E-22"
-        iyy="4.3309E-06"
-        iyz="-1.1353E-21"
-        izz="5.4641E-06" />
-    </inertial>
-    <visual>
-      <origin
-        xyz="0 0 0"
-        rpy="0 0 0" />
-      <geometry>
-        <mesh
-          filename="package://r2b_env/meshes/box_top.STL" />
-      </geometry>
-      <material
-        name="">
-        <color
-          rgba="0.79216 0.81961 0.93333 1" />
-      </material>
-    </visual>
-    <collision>
-      <origin
-        xyz="0 0 0"
-        rpy="0 0 0" />
-      <geometry>
-        <mesh
-          filename="package://r2b_env/meshes/box_top.STL" />
-      </geometry>
-    </collision>
-  </link>
-  <joint
-    name="box_top_jnt"
-    type="fixed">
-    <origin
-      xyz="-0.146 0.12875 -0.034071"
-      rpy="0 0 0" />
-    <parent
-      link="upper_compartment" />
-    <child
-      link="box_top" />
-    <axis
-      xyz="0 0 0" />
-  </joint>
-  <link
-    name="box_mid">
-    <inertial>
-      <origin
-        xyz="-0.015 -1.3878E-17 1.3878E-17"
-        rpy="0 0 0" />
-      <mass
-        value="0.031755" />
-      <inertia
-        ixx="5.751E-06"
-        ixy="3.3449E-21"
-        ixz="5.6808E-23"
-        iyy="4.6071E-06"
-        iyz="-5.1228E-22"
-        izz="5.9071E-06" />
-    </inertial>
-    <visual>
-      <origin
-        xyz="0 0 0"
-        rpy="0 0 0" />
-      <geometry>
-        <mesh
-          filename="package://r2b_env/meshes/box_mid.STL" />
-      </geometry>
-      <material
-        name="">
-        <color
-          rgba="0.79216 0.81961 0.93333 1" />
-      </material>
-    </visual>
-    <collision>
-      <origin
-        xyz="0 0 0"
-        rpy="0 0 0" />
-      <geometry>
-        <mesh
-          filename="package://r2b_env/meshes/box_mid.STL" />
-      </geometry>
-    </collision>
-  </link>
-  <joint
-    name="box_mid_jnt"
-    type="fixed">
-    <origin
-      xyz="-0.146 0.08925 -0.033821"
-      rpy="0 0 0" />
-    <parent
-      link="upper_compartment" />
-    <child
-      link="box_mid" />
-    <axis
-      xyz="0 0 0" />
-  </joint>
-  <link
-    name="box_down">
-    <inertial>
-      <origin
-        xyz="-0.015 1.3878E-17 1.3878E-17"
-        rpy="0 0 0" />
-      <mass
-        value="0.030885" />
-      <inertia
-        ixx="5.4081E-06"
-        ixy="1.8055E-21"
-        ixz="1.3388E-21"
-        iyy="4.4809E-06"
-        iyz="4.7747E-22"
-        izz="5.5599E-06" />
-    </inertial>
-    <visual>
-      <origin
-        xyz="0 0 0"
-        rpy="0 0 0" />
-      <geometry>
-        <mesh
-          filename="package://r2b_env/meshes/box_down.STL" />
-      </geometry>
-      <material
-        name="">
-        <color
-          rgba="0.79216 0.81961 0.93333 1" />
-      </material>
-    </visual>
-    <collision>
-      <origin
-        xyz="0 0 0"
-        rpy="0 0 0" />
-      <geometry>
-        <mesh
-          filename="package://r2b_env/meshes/box_down.STL" />
-      </geometry>
-    </collision>
-  </link>
-  <joint
-    name="box_down_jnt"
-    type="fixed">
-    <origin
-      xyz="-0.146 0.04975 -0.033821"
-      rpy="0 0 0" />
-    <parent
-      link="upper_compartment" />
-    <child
-      link="box_down" />
-    <axis
-      xyz="0 0 0" />
-  </joint> -->
+  <gazebo>
+    <static>true</static>
+  </gazebo>
 </robot>

Commit message: Modified compartment spawning

File: r2b_env/urdf/compartments.urdf.xacro (robot description, xacro)
@@ -42,5 +42,5 @@
   </link>
   <joint name="fixed" type="fixed">
-		<origin xyz="0.0 0.0 0.0" rpy="0.0 0.0 0.0"/>
+		<origin xyz="0.0 0.0 0.0" rpy="1.5708 0.0 0.0"/>
 		<parent link="world"/>
 		<child link="lower_compartment"/>
